File: kicad/boards_version_2/stack_data_v2/stack_data_v2.kicad_sch (KiCad schematic)
At the start: 23 parts

Commit message: Started work on stack sequencer in kicad
Parts:
- removed U11: ~, Package_DIP:DIP-28_W15.24mm, symbol custom_symbol_lib:32Kx8_sram
- removed U17: ~, Package_DIP:DIP-16_W7.62mm, symbol custom_symbol_lib:4bit_adder
- removed U18: ~, Package_DIP:DIP-20_W7.62mm, symbol custom_symbol_lib:rising_edge_8_bit_latch
- removed U22, U23: ~, Package_DIP:DIP-16_W7.62mm, symbol custom_symbol_lib:2x4_bit_multiplexer
- added U11: ~, Package_DIP:DIP-16_W7.62mm, symbol custom_symbol_lib:4bit_adder
- added U13, U19: ~, Package_DIP:DIP-16_W7.62mm, symbol custom_symbol_lib:2x4_bit_multiplexer
- added U17: ~, Package_DIP:DIP-20_W7.62mm, symbol custom_symbol_lib:rising_edge_8_bit_latch
- added U22: ~, Package_DIP:DIP-28_W15.24mm, symbol custom_symbol_lib:32Kx8_sram
Connections:
- net at U1.7 (C_IN), U1.8 (GND), U10.11 (I4)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: now also U11.8 (GND), U13.15 (OE#), U13.8 (GND), U17.1 (OE#), U17.10 (GND), U19.15 (OE#), U19.8 (GND), U22.14 (GND), U22.20 (CE#)
- net at U5.20 (Offset_latch_CLK), U9.11 (CLK): now also U12.11 (CLK)
- net at U48.27 (D7), U9.12 (Q7), U9.9 (D7): now also U12.9 (D7), U22.19 (D7)
- net at U48.26 (D6), U9.13 (Q6), U9.8 (D6): now also U12.8 (D6), U22.18 (D6)
- net at U48.25 (D5), U9.14 (Q5), U9.7 (D5): now also U12.7 (D5), U22.17 (D5)
- net at U48.24 (D4), U9.15 (Q4), U9.6 (D4): now also U12.6 (D4), U22.16 (D4)
- net at U48.23 (D3), U9.16 (Q3), U9.5 (D3): now also U12.5 (D3), U22.15 (D3)
- net at U48.22 (D2), U9.17 (Q2), U9.4 (D2): now also U12.4 (D2), U22.13 (D2)
- net at U48.21 (D1), U9.18 (Q1), U9.3 (D1): now also U12.3 (D1), U22.12 (D1)
- net at U48.20 (D0), U9.19 (Q0), U9.2 (D0): now also U12.2 (D0), U22.11 (D0)
- net at U1.16 (V+), U1.6 (B0), U10.14 (V+)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: now also U15.11 (B3), U15.15 (B2), U15.2 (B1), U15.6 (B0), U11.16 (V+), U11.7 (C_IN), U13.16 (V+), U17.20 (V+), U19.16 (V+), U22.28 (V+); no longer U14.7 (C_IN)
- net at U5.16 (Post-adder_latch_CLK), U6.11 (CLK): now also U17.11 (CLK); no longer U7.11 (CLK)
- net at U20.1 (S), U21.1 (S), U5.19 (ToS_(0)_/_Offset_(1)_select): now also U13.1 (S), U19.1 (S)
- net at U5.22 (Pre-adder_latch_CLK), U8.11 (CLK): now also U7.11 (CLK); no longer U12.11 (CLK)
- net at U12.12 (Q7): now also U14.11 (B3); no longer U4.12 (A3)
- net at U12.13 (Q6): now also U14.15 (B2); no longer U4.14 (A2)
- net at U12.14 (Q5): now also U14.2 (B1); no longer U4.3 (A1)
- net at U12.15 (Q4): now also U14.6 (B0); no longer U4.5 (A0)
- net at U3.12 (A3): now also U7.16 (Q3); no longer U12.16 (Q3)
- net at U3.14 (A2): now also U7.17 (Q2); no longer U12.17 (Q2)
- net at U3.3 (A1): now also U7.18 (Q1); no longer U12.18 (Q1)
- net at U3.5 (A0): now also U7.19 (Q0); no longer U12.19 (Q0)
- net at U7.15 (Q4): now also U4.5 (A0); no longer U12.6 (D4)
- net at U7.14 (Q5): now also U4.3 (A1); no longer U12.7 (D5)
- net at U7.13 (Q6): now also U4.14 (A2); no longer U12.8 (D6)
- net at U7.12 (Q7): now also U4.12 (A3); no longer U12.9 (D7)
- net at U7.7 (D5): now also U16.3 (A1), U6.14 (Q5), U13.5 (A1); no longer U4.1 (Σ1)
- net at U7.9 (D7): now also U16.12 (A3), U6.12 (Q7), U13.14 (A3); no longer U4.10 (Σ3)
- net at U7.8 (D6): now also U16.14 (A2), U6.13 (Q6), U13.11 (A2); no longer U4.13 (Σ2)
- net at U7.6 (D4): now also U16.5 (A0), U6.15 (Q4), U13.2 (A0); no longer U4.4 (Σ0)
- net at U4.7 (C_IN): now also U3.9 (C_OUT)
- net at U20.4 (Q0): now also U33.5 (4), U22.6 (A4); no longer U33.1 (0)
- net at U33.10 (9): now also U19.7 (Q1), U22.24 (A9)
- net at U33.11 (10): now also U19.9 (Q2), U22.21 (A10)
- net at U33.12 (11): now also U19.12 (Q3), U22.23 (A11)
- net at U33.13 (12): now also U13.4 (Q0), U22.2 (A12)
- net at U33.14 (13): now also U13.7 (Q1), U22.26 (A13)
- net at U33.15 (14): now also U13.9 (Q2), U22.1 (A14)
- net at U33.16 (15): now also U13.12 (Q3)
- net at U20.7 (Q1): now also U33.6 (5), U22.5 (A5); no longer U33.2 (1)
- net at U20.9 (Q2): now also U33.7 (6), U22.4 (A6); no longer U33.3 (2)
- net at U20.12 (Q3): now also U33.8 (7), U22.3 (A7); no longer U33.4 (3)
- net at U21.4 (Q0): now also U33.1 (0), U22.10 (A0); no longer U33.5 (4)
- net at U21.7 (Q1): now also U33.2 (1), U22.9 (A1); no longer U33.6 (5)
- net at U21.9 (Q2): now also U33.3 (2), U22.8 (A2); no longer U33.7 (6)
- net at U21.12 (Q3): now also U33.4 (3), U22.7 (A3); no longer U33.8 (7)
- net at U33.9 (8): now also U19.4 (Q0), U22.25 (A8)
- net at U14.14 (A2), U20.11 (A2): now also U8.8 (D6), U17.13 (Q6); no longer U6.17 (Q2), U8.4 (D2)
- net at U14.12 (A3), U20.14 (A3): now also U8.9 (D7), U17.12 (Q7); no longer U6.16 (Q3), U8.5 (D3)
- net at U14.5 (A0), U20.2 (A0): now also U8.6 (D4), U17.15 (Q4); no longer U6.19 (Q0), U8.2 (D0)
- net at U14.3 (A1), U20.5 (A1): now also U8.7 (D5), U17.14 (Q5); no longer U6.18 (Q1), U8.3 (D1)
- net at U3.1 (Σ1): now also U6.3 (D1); no longer U7.3 (D1)
- net at U3.10 (Σ3): now also U6.5 (D3); no longer U7.5 (D3)
- net at U3.13 (Σ2): now also U6.4 (D2); no longer U7.4 (D2)
- net at U3.4 (Σ0): now also U6.2 (D0); no longer U7.2 (D0)
- net at U2.1 (Σ1): now also U17.7 (D5); no longer U6.7 (D5)
- net at U2.10 (Σ3): now also U17.9 (D7); no longer U6.9 (D7)
- net at U2.13 (Σ2): now also U17.8 (D6); no longer U6.8 (D6)
- net at U2.4 (Σ0): now also U17.6 (D4); no longer U6.6 (D4)
- net at U10.2 (O0): now also U22.22 (OE#)
- net at U10.4 (O1): now also U22.27 (WE#)
- net at U1.1 (Σ1): now also U17.3 (D1); no longer U6.3 (D1)
- net at U1.10 (Σ3): now also U17.5 (D3); no longer U6.5 (D3)
- net at U1.13 (Σ2): now also U17.4 (D2); no longer U6.4 (D2)
- net at U1.4 (Σ0): now also U17.2 (D0); no longer U6.2 (D0)
- net at U21.6 (B1): now also U11.1 (Σ1); no longer U15.1 (Σ1)
- net at U21.13 (B3): now also U11.10 (Σ3); no longer U15.10 (Σ3)
- net at U21.10 (B2): now also U11.13 (Σ2); no longer U15.13 (Σ2)
- net at U21.3 (B0): now also U11.4 (Σ0); no longer U15.4 (Σ0)
- net at U16.13 (Σ2): now also U13.10 (B2)
- net at U16.10 (Σ3): now also U13.13 (B3)
- net at U16.4 (Σ0): now also U13.3 (B0)
- net at U16.1 (Σ1): now also U13.6 (B1)
- new net: U11.9 (C_OUT), U14.7 (C_IN)
- new net: U11.5 (A0), U17.19 (Q0), U21.2 (A0), U8.2 (D0)
- new net: U11.3 (A1), U17.18 (Q1), U21.5 (A1), U8.3 (D1)
- new net: U11.14 (A2), U17.17 (Q2), U21.11 (A2), U8.4 (D2)
- new net: U11.12 (A3), U17.16 (Q3), U21.14 (A3), U8.5 (D3)
- new net: U15.5 (A0), U19.2 (A0), U6.19 (Q0), U7.2 (D0)
- new net: U15.3 (A1), U19.5 (A1), U6.18 (Q1), U7.3 (D1)
- new net: U15.14 (A2), U19.11 (A2), U6.17 (Q2), U7.4 (D2)
- new net: U15.12 (A3), U19.14 (A3), U6.16 (Q3), U7.5 (D3)
- new net: U15.1 (Σ1), U19.6 (B1)
- new net: U15.10 (Σ3), U19.13 (B3)
- new net: U15.13 (Σ2), U19.10 (B2)
- new net: U15.4 (Σ0), U19.3 (B0)
- new net: U4.4 (Σ0), U6.6 (D4)
- new net: U4.1 (Σ1), U6.7 (D5)
- new net: U4.13 (Σ2), U6.8 (D6)
- new net: U4.10 (Σ3), U6.9 (D7)
- new net: U11.11 (B3), U12.16 (Q3)
- new net: U11.15 (B2), U12.17 (Q2)
- new net: U11.2 (B1), U12.18 (Q1)
- new net: U11.6 (B0), U12.19 (Q0)
